Commit message: 자율 매핑을 하이브리드 탐색 구조와 안정적인 TF/SLAM 기준으로 재설계한다
LiDAR 기반 자율 매핑이 시작점에서 멈추거나 좁은 구역에서 회전 루프에 빠지던 문제를 줄이기 위해 탐색 supervisor, SLAM, TF, Nav2 recovery 구성을 함께 리팩토링했다.

- frontier explorer를 bootstrap 직진, boundary follow, frontier explore, recovery, coverage fill 상태를 가진 상위 supervisor로 재구성
- 센서 TF 기준을 URDF와 Gazebo SDF에 맞춰 정리하고 중복 static TF 발행 제거
- 매핑 세션에서는 raw odom TF를 SLAM 기준으로 사용하고 EKF는 filtered odometry 토픽만 발행하도록 분리
- slam_toolbox를 sync 모드와 TF restamp 기준으로 조정해 map TF 생성 기준선 복구
- collision monitor lifecycle과 cmd_vel 경로를 정리해 bootstrap 직진 명령이 실제 로봇 이동으로 이어지도록 수정
- Nav2 매핑 파라미터와 recovery BT를 직진 우선, 확실한 탈출 중심으로 재튜닝
- 관련 테스트와 매핑 스모크 검증을 다시 맞춤

File: agribot_ws/src/agribot_description/urdf/agribot.urdf (robot description, URDF)
Before this commit: robot agribot, 7 links, 6 joints
Joints:
- joint camera_joint: origin xyz=0.2 0 0.1 rpy=0 0 0 -> xyz=0.2 0 0.3 rpy=0 0 0
- joint imu_joint: origin xyz=0 0 0.05 rpy=0 0 0 -> xyz=0 0 0.25 rpy=0 0 0
- joint lidar_joint: origin xyz=0 0 0.15 rpy=0 0 0 -> xyz=0 0 0.35 rpy=0 0 0

Commit message: S14P21A602-94 맵, 로봇, 스프링클러 추가

File: agribot_ws/src/agribot_description/urdf/agribot.urdf (robot description, URDF)
Before this commit: robot agribot, 7 links, 6 joints
Links:
- link base_link: geometry collision box size=0.4 0.3 0.15; visual mesh filename=package://agribot_description/models/agribot/meshes/agribot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 scale=0.14 0.14 0.14

Commit message: 수확 팔과 바구니 모델을 추가한다

File: agribot_ws/src/agribot_description/urdf/agribot.urdf (robot description, URDF)
Before this commit: robot agribot, 7 links, 6 joints
Links:
- added link harvest_arm_link, mass 0.8; collision box size=0.02 0.014 0.10; collision box size=0.02 0.014 0.10
- added link harvest_basket_link, mass 0.5; collision box size=0.02 0.14 0.12; collision box size=0.02 0.14 0.12
Joints:
- added joint harvest_arm_joint: type fixed, parent base_link, child harvest_arm_link, origin xyz=-0.02 0 0.22 rpy=0 0 0
- added joint harvest_basket_joint: type fixed, parent base_link, child harvest_basket_link, origin xyz=-0.14 0 0.20 rpy=0 0 0

Commit message: [S14P21A602-137] Gazebo 수확 시뮬레이션과 안전 종료 로직만 dev2에 선별 반영
feature/S14P21A602-137 전체를 합치지 않고, Gazebo 수확 시뮬레이션 강화, 로봇 모델·월드·state bridge 자산, shutdown cleanup 개선 범위만 dev2에 선별 반영했다.

또한 branch merge로는 들어오지 않는 startup_map_tf_broadcaster.py를 dev2 문맥에 맞게 직접 수정해, /amcl_pose 수신 이후 임시 identity map->odom broadcaster가 계속 남지 않도록 정리했다.

신규로 추가된 Python·YAML·테스트 파일에는 팀원이 역할을 빠르게 이해할 수 있도록 한글 설명 주석을 보강했다.

File: agribot_ws/src/agribot_description/urdf/agribot.urdf (robot description, URDF)
Before this commit: robot agribot, 9 links, 8 joints
Joints:
- joint harvest_arm_joint: axis (none) -> 0 1 0; limit (none) -> lower=-0.60 upper=0.70 effort=10.0 velocity=1.5; origin xyz=-0.02 0 0.22 rpy=0 0 0 -> xyz=0.04 0 0.29 rpy=0 0.15 0; type fixed -> revolute

Commit message: 로봇 바퀴와 캐스터 visual을 반투명 바퀴 표현으로 조정
Gazebo에서 로봇 전면 하단의 캐스터가 작은 토마토처럼 보이는 혼동을 줄이기 위해, 바퀴와 캐스터 visual 표현을 정리했다.

메인 구동 바퀴는 기존 원통형 바퀴 형태를 유지하되 투명도 25%로 맞췄고, 캐스터는 sphere visual을 작은 cylinder visual로 바꿔 실제 바퀴처럼 보이게 했다. 카메라 visual도 같은 반투명 정책을 적용해 화면에서 덜 튀도록 조정했다.

이번 변경은 visual만 수정한 것이므로 센서 토픽, 충돌, 주행 물리는 그대로 유지된다. 또한 model.sdf와 urdf 파일에는 다른 에이전트가 수정 중인 로봇팔 hunk가 함께 있었기 때문에, 이번 커밋은 바퀴/캐스터/카메라 visual 관련 변경만 분리해서 담았다.

File: agribot_ws/src/agribot_description/urdf/agribot.urdf (robot description, URDF)
Before this commit: robot agribot, 9 links, 8 joints
Links:
- link caster: geometry collision sphere radius=0.03; visual cylinder length=0.018 radius=0.028

Commit message: 최종 시연용 관측 접근 보완과 Gazebo 자산 정렬을 마무리
- 울타리 근처 최종 관측 지점으로 바로 갈 수 없을 때 중간 대체 후보를 순차 탐색하도록 수동 명령 실행기를 보강했습니다.
- route의 lane_side에 따라 지도 표시용 접근 거리와 측면 한계를 다르게 계산하도록 backend와 순찰 설정을 확장했습니다.
- 로봇팔이 상하 반전되어 보이던 문제를 SDF와 URDF에서 함께 바로잡고, 충돌체 방향도 동일 기준으로 정렬했습니다.
- 토마토 모델의 재질 표현과 자산 테스트를 현재 Gazebo 자산 기준으로 맞춰 시연 화면 품질을 안정화했습니다.
- 시연 명령어 문서와 트러블슈팅 문서를 보강해 팀원이 pull 받은 뒤에도 같은 절차로 실행하고 회고할 수 있게 정리했습니다.

검증:
- python3 -m pytest agribot_ws/src/agribot_bringup/test/test_robot_manual_command_executor.py
- python3 -m pytest agribot_ws/src/agribot_description/test/test_world_assets.py

File: agribot_ws/src/agribot_description/urdf/agribot.urdf (robot description, URDF)
Before this commit: robot agribot, 9 links, 8 joints
Joints:
- joint harvest_arm_joint: origin xyz=0.04 0 0.29 rpy=0 0.15 0 -> xyz=0.04 0 0.48 rpy=-3.1416 0 0
